File: PCB/code of claw translator/code of claw translator.kicad_sch (KiCad schematic)
At the start: 22 parts, among them J1 Conn_01x20_Socket, J10 Conn_01x01_Socket, J11 Conn_01x03_Socket, J2 Conn_01x20_Socket, J3 Conn_01x14_Socket, J4 Conn_01x08_Socket, J5 Conn_01x08_Socket, J6 Conn_01x06_Socket, J7 Conn_01x01_Socket, J8 Conn_01x01_Socket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

Commit message: Designing rough draft of final look
Parts:
- removed SW1, SW2, SW3, SW4, SW5, SW6, SW7: SW_Push_Dual, symbol Switch:SW_Push_Dual
- added J12, J13, J14, J15, J16, J17, J18, J19, J20, J21, J22, J23, J24, J25, J26, J27: Conn_01x01_Socket, Connector_PinSocket_2.54mm:PinSocket_1x01_P2.54mm_Vertical, symbol Connector:Conn_01x01_Socket
- added J32, J33, J34, J35, J36, J37, J38, J39, J40, J41, J42, J43: Conn_01x01_Socket, Connector_PinSocket_2.54mm:PinSocket_1x01_P2.54mm_Horizontal, symbol Connector:Conn_01x01_Socket
Connections:
- net A10: now also J34.1 (Pin_1)
- net A11: now also J26.1 (Pin_1)
- net A12: now also J18.1 (Pin_1)
- net A8: now also J38.1 (Pin_1)
- net A9: now also J42.1 (Pin_1)
- net B1: now also J14.1 (Pin_1)
- net B13: now also J22.1 (Pin_1)
- net GND: now also J12.1 (Pin_1), J16.1 (Pin_1), J20.1 (Pin_1), J24.1 (Pin_1), J32.1 (Pin_1), J36.1 (Pin_1), J40.1 (Pin_1)
Other:
- note added: "Backspace button"
- note added: "Clear button"
- note added: "Click button"
- note added: "Period button"
- note added: "Scratch button"
- note added: "Space button"
- note added: "Tap button"
- note removed: "Backspace"
- note removed: "Clear"
- note removed: "Click"
- note removed: "Period"
- note removed: "Scratch"
- note removed: "Space"
- note removed: "Tap"
- moved on the sheet: J3
